File: Hardware/aircraft.kicad_sch (KiCad schematic)
At the start: 0 parts

Commit message: version 0.1.0
Other:
- removed sheet Programming_Debug
- note added: "Gravitum Flight Control System"
- note added: "Version 0.1.0"
Changed lines of the file:
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@@
 	(title_block
 		(title "Gravitum Flight Control System")
+		(rev "0.1.0")
 		(company "Breno Soares Alves")
 	)
-	(sheet
-		(at 152.4 43.18)
+	(text "Gravitum Flight Control System"
+		(exclude_from_sim no)
+		(at 152.4 39.878 0)
+		(effects
+			(font
+				(size 6.35 6.35)
+				(thickness 1.27)
+				(bold yes)
+				(italic yes)
+			)
+		)
+	)
+	(text "Version 0.1.0"
+		(exclude_from_sim no)
+		(at 149.098 51.562 0)
+		(effects
+			(font
+				(size 2.54 2.54)
+			)
+		)
+	)
+	(sheet
+		(at 173.99 67.31)
 		(size 30.48 27.94)
 		(exclude_from_sim no)
@@
 		)
 		(property "Sheetname" "Navigation_Peripherals"
-			(at 152.4 42.4684 0)
+			(at 173.99 66.5984 0)
 			(effects
 				(font
@@
 		)
 		(property "Sheetfile" "navigation_peripherals.kicad_sch"
-			(at 152.4 71.7046 0)
+			(at 173.99 95.8346 0)
 			(effects
 				(font
@@
 	)
 	(sheet
-		(at 152.4 78.74)
+		(at 134.62 102.87)
 		(size 30.48 27.94)
 		(exclude_from_sim no)
@@
 		)
 		(property "Sheetname" "Flight_Control_Peripherals"
-			(at 152.4 78.0284 0)
+			(at 134.62 102.1584 0)
 			(effects
 				(font
@@
 		)
 		(property "Sheetfile" "flight_control_peripherals.kicad_sch"
-			(at 152.4 107.2646 0)
+			(at 134.62 131.3946 0)
 			(effects
 				(font
@@
 	)
 	(sheet
-		(at 73.66 43.18)
+		(at 95.25 67.31)
 		(size 30.48 27.94)
 		(exclude_from_sim no)
@@
 		)
 		(property "Sheetname" "Power_Supply"
-			(at 73.66 42.4684 0)
+			(at 95.25 66.5984 0)
 			(effects
 				(font
@@
 		)
 		(property "Sheetfile" "power_supply.kicad_sch"
-			(at 73.66 71.7046 0)
+			(at 95.25 95.8346 0)
 			(effects
 				(font
@@
 	)
 	(sheet
-		(at 73.66 78.74)
-		(size 30.48 27.94)
-		(exclude_from_sim no)
-		(in_bom yes)
-		(on_board yes)
-		(dnp no)
-		(fields_autoplaced yes)
-		(stroke
-			(width 0.1524)
-			(type solid)
-		)
-		(fill
-			(color 0 0 0 0.0000)
-		)
-		(property "Sheetname" "Programming_Debug"
-			(at 73.66 78.0284 0)
-			(effects
-				(font
-					(size 1.27 1.27)
-				)
-				(justify left bottom)
-			)
-		)
-		(property "Sheetfile" "programming_debug.kicad_sch"
-			(at 73.66 107.2646 0)
+		(at 95.25 102.87)
+		(size 30.48 27.94)
+		(exclude_from_sim no)
+		(in_bom yes)
+		(on_board yes)
+		(dnp no)
+		(fields_autoplaced yes)
+		(stroke
+			(width 0.1524)
+			(type solid)
+		)
+		(fill
+			(color 0 0 0 0.0000)
+		)
+		(property "Sheetname" "Flight_Control_Unit"
+			(at 95.25 102.1584 0)
+			(effects
+				(font
+					(size 1.27 1.27)
+				)
+				(justify left bottom)
+			)
+		)
+		(property "Sheetfile" "flight_control_unit.kicad_sch"
+			(at 95.25 131.3946 0)
+			(effects
+				(font
+					(size 1.27 1.27)
+				)
+				(justify left top)
+			)
+		)
+		(instances
+			(project "aircraft"
+				(path "/8dc22ddc-eb0a-4b80-a714-26a959e826d2"
+					(page "5")
+				)
+			)
+		)
+	)
+	(sheet
+		(at 173.99 102.87)
+		(size 30.48 27.94)
+		(exclude_from_sim no)
+		(in_bom yes)
+		(on_board yes)
+		(dnp no)
+		(fields_autoplaced yes)
+		(stroke
+			(width 0.1524)
+			(type solid)
+		)
+		(fill
+			(color 0 0 0 0.0000)
+		)
+		(property "Sheetname" "Other_Connections"
+			(at 173.99 102.1584 0)
+			(effects
+				(font
+					(size 1.27 1.27)
+				)
+				(justify left bottom)
+			)
+		)
+		(property "Sheetfile" "other_connections.kicad_sch"
+			(at 173.99 131.3946 0)
 			(effects
 				(font
@@
 	)
 	(sheet
-		(at 113.03 78.74)
-		(size 30.48 27.94)
-		(exclude_from_sim no)
-		(in_bom yes)
-		(on_board yes)
-		(dnp no)
-		(fields_autoplaced yes)
-		(stroke
-			(width 0.1524)
-			(type solid)
-		)
-		(fill
-			(color 0 0 0 0.0000)
-		)
-		(property "Sheetname" "Flight_Control_Unit"
-			(at 113.03 78.0284 0)
-			(effects
-				(font
-					(size 1.27 1.27)
-				)
-				(justify left bottom)
-			)
-		)
-		(property "Sheetfile" "flight_control_unit.kicad_sch"
-			(at 113.03 107.2646 0)
-			(effects
-				(font
-					(size 1.27 1.27)
-				)
-				(justify left top)
-			)
-		)
-		(instances
-			(project "aircraft"
-				(path "/8dc22ddc-eb0a-4b80-a714-26a959e826d2"
-					(page "5")
-				)
-			)
-		)
-	)
-	(sheet
-		(at 191.77 43.18)
-		(size 30.48 27.94)
-		(exclude_from_sim no)
-		(in_bom yes)
-		(on_board yes)
-		(dnp no)
-		(fields_autoplaced yes)
-		(stroke
-			(width 0.1524)
-			(type solid)
-		)
-		(fill
-			(color 0 0 0 0.0000)
-		)
-		(property "Sheetname" "Other_Connections"
-			(at 191.77 42.4684 0)
-			(effects
-				(font
-					(size 1.27 1.27)
-				)
-				(justify left bottom)
-			)
-		)
-		(property "Sheetfile" "other_connections.kicad_sch"
-			(at 191.77 71.7046 0)
-			(effects
-				(font
-					(size 1.27 1.27)
-				)
-				(justify left top)
-			)
-		)
-		(instances
-			(project "aircraft"
-				(path "/8dc22ddc-eb0a-4b80-a714-26a959e826d2"
-					(page "8")
-				)
-			)
-		)
-	)
-	(sheet
-		(at 113.03 43.18)
+		(at 134.62 67.31)
 		(size 30.48 27.94)
 		(exclude_from_sim no)
@@
 		)
 		(property "Sheetname" "Navigation_Unit"
-			(at 113.03 42.4684 0)
+			(at 134.62 66.5984 0)
 			(effects
 				(font
@@
 		)
 		(property "Sheetfile" "navigation_unit.kicad_sch"
-			(at 113.03 71.7046 0)
-			(effects
-				(font
+			(at 134.62 95.8346 0)
+			(effects
+				(font

Commit message: i forgot to change the damn label
Other:
- note added: "Version 0.1.1"
- note removed: "Version 0.1.0"
Changed lines of the file:
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@@
 		)
 	)
-	(text "Version 0.1.0"
+	(text "Version 0.1.1"
 		(exclude_from_sim no)
 		(at 149.098 51.562 0)
