File: Hardware/navigation_peripherals.kicad_sch (KiCad schematic)
At the start: 29 parts, among them J2 5-1814832-1, J3 Conn_01x04, J5 Conn_01x04, U10 BMP390, U11 W25N01GVZEIG_TR, U5 IST8310, U6 NEO-M8N, U7 BMI088, U8 TMP100, U9 24CW1280T-I/OT

Commit message: firmware started, freertos, initial sensors abstractions, some pin layout changes
Parts:
- U10: footprint 10LGA_2X2X0p75_BOS -> (none)
- U9: footprint SOT-23-5_2P9X1P6_MCH -> (none)
Changed lines of the file:
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@@
 			)
 		)
-		(property "Footprint" "10LGA_2X2X0p75_BOS"
+		(property "Footprint" ""
 			(at 212.09 41.91 0)
 			(effects
@@
 			)
 		)
-		(property "Footprint" "SOT-23-5_2P9X1P6_MCH"
+		(property "Footprint" ""
 			(at 208.28 85.09 0)
 			(effects

Commit message: add some footprints, and pcb configs
Parts:
- C30, C31, C34, C35, C36, C37, C38, C39: footprint (none) -> Capacitor_SMD:C_0603_1608Metric
- U10: footprint (none) -> Aircraft_Footprints:10LGA_2X2X0p75_BOS
- U9: footprint (none) -> Aircraft_Footprints:SOT-23-5_2P9X1P6_MCH
- renumbered J5 to J4, R21 to R19, R22 to R20, R23 to R21, R24 to R22
