File: Hardware/other_connections.kicad_sch (KiCad schematic)
At the start: 42 parts, among them J13 Conn_01x02, J14 Conn_02x05_Odd_Even, J15 Conn_02x05_Odd_Even, J16 USB_B_Micro, J17 USB_B_Micro, J18 USB_B_Micro, J19 USB_B_Micro, U16 CH330N, U17 CH330N

Commit message: add some footprints, and pcb configs
Parts:
- added JP4: SolderJumper_2_Open, symbol Jumper:SolderJumper_2_Open
- added R48, R52: 560, Resistor_SMD:R_0603_1608Metric, symbol Device:R
- C60, C61, C62, C63: footprint (none) -> Capacitor_SMD:C_0603_1608Metric
- D12: footprint (none) -> Diode_SMD:D_SOD-323_HandSoldering
- D13: renamed from D16; footprint (none) -> Diode_SMD:D_SOD-323_HandSoldering
- D14: renamed from D13; footprint (none) -> LED_SMD:LED_0603_1608Metric
- D15: renamed from D14; footprint (none) -> Diode_SMD:D_SOD-323_HandSoldering
- D16: renamed from D17; footprint (none) -> Diode_SMD:D_SOD-323_HandSoldering
- D17: renamed from D15; footprint (none) -> LED_SMD:LED_0603_1608Metric
- FB3, FB6: footprint (none) -> Inductor_SMD:L_0805_2012Metric
- FB4: renamed from FB5; footprint (none) -> Inductor_SMD:L_0805_2012Metric
- FB5: renamed from FB4; footprint (none) -> Inductor_SMD:L_0805_2012Metric
- R35: renamed from R46; footprint (none) -> Resistor_SMD:R_0603_1608Metric_Pad0.98x0.95mm_HandSolder
- R36: renamed from R47; footprint (none) -> Resistor_SMD:R_0603_1608Metric_Pad0.98x0.95mm_HandSolder
- R37: renamed from R48; footprint (none) -> Resistor_SMD:R_0603_1608Metric
- R38: renamed from R49; footprint (none) -> Resistor_SMD:R_0603_1608Metric
- R39, R40, R41, R42, R43, R44, R45: footprint (none) -> Resistor_SMD:R_0603_1608Metric
- R46: renamed from R35; footprint (none) -> Resistor_SMD:R_0603_1608Metric
- R47: renamed from R36; footprint (none) -> Resistor_SMD:R_0603_1608Metric
- R49: renamed from R50; footprint (none) -> Resistor_SMD:R_0603_1608Metric_Pad0.98x0.95mm_HandSolder
- R50: renamed from R52; footprint (none) -> Resistor_SMD:R_0603_1608Metric
- R51: renamed from R53; footprint (none) -> Resistor_SMD:R_0603_1608Metric
- R53: renamed from R51; footprint (none) -> Resistor_SMD:R_0603_1608Metric_Pad0.98x0.95mm_HandSolder
- renumbered J14 to J12, J16 to J14, J18 to J16, J19 to J18
Connections:
- net GND: now also J16.5 (GND), J16.6 (Shield), J18.5 (GND), J18.6 (Shield)
- net at D16.2 (A), J18.1 (VBUS): now also JP4.1 (A)
- net at J18.4 (ID): now also R52.1
- net at J16.4 (ID): now also R48.1
- new net FCU_USB_OTG_FS_ID: R48.2
- new net NU_USB_OTG_FS_ID: R52.2
- new net NU_USB_OTG_FS_VBUS: JP4.2 (B)
- no-connect marks 14 -> 10
Other:
- note removed: "NU don't have VBUS because of pin assignment, that is not a problem because VBUS isn't required to run Device Mode"
- moved on the sheet: D16, FB6, J18, R50, R51
