File: Hardware/aircraft.kicad_pcb (KiCad board)
At the start: 4 copper layers, 106.1 x 55 mm, 194 parts, among them J1 Conn_01x02_Pin, J10 Conn_01x06, J12 Conn_02x05_Odd_Even, J13 Conn_01x02, J14 USB_B_Micro, J15 Conn_02x05_Odd_Even, J16 USB_B_Micro, J17 USB_B_Micro, J18 USB_B_Micro, J19 U.FL-R-SMT-1_80_, J2 DM3AT-SF-PEJM5, J3 Conn_01x04, J4 Conn_01x04, J5 Conn_01x10, J6 Conn_02x10_Odd_Even, J7 Conn_01x04, J8 Conn_01x04, J9 Conn_02x06_Odd_Even, SW1 SW_SPDT, SW2 SW_Push_Dual, SW3 SW_SPDT, SW4 SW_Push_Dual, U1 MIC26903YJL-TR, U10 BMP390, U11 W25N01GVZEIG_TR, U12 STM32F405RGTx, U13 W25N01GVZEIG_TR, U14 24CW1280T-I/OT, U15 PCA9685PW_118, U16 CH330N, U17 CH330N, U2 LD39200PU33R, U3 INA226, U4 STM32F405RGTx, U5 IST8310, U6 NEO-M8N, U7 BMI088, U8 TMP100, U9 24CW1280T-I/OT, Y1 25MHz, Y2 25MHz

Commit message: hardware: reorganizing components, im fucked
Parts:
- removed G*** (x2): LOGO, LOGO
- removed the REF** at (198.6, 126.7)
- removed the REF** at (102.6, 126.7)
- removed the REF** at (198.6, 81.7)
- removed the REF** at (102.6, 81.7)
- added REF**: MountingHole_2.2mm_M2_Pad_Via, MountingHole:MountingHole_2.2mm_M2_Pad_Via, F.Cu at (245.0, 145.0)
- added REF**: MountingHole_2.2mm_M2_Pad_Via, MountingHole:MountingHole_2.2mm_M2_Pad_Via, F.Cu at (155.0, 145.0)
- added REF**: MountingHole_2.2mm_M2_Pad_Via, MountingHole:MountingHole_2.2mm_M2_Pad_Via, F.Cu at (245.0, 105.0)
- added REF**: MountingHole_2.2mm_M2_Pad_Via, MountingHole:MountingHole_2.2mm_M2_Pad_Via, F.Cu at (155.0, 105.0)
- C11, C2: footprint Capacitor_SMD:C_1206_3216Metric_Pad1.33x1.80mm_HandSolder -> Capacitor_SMD:C_1206_3216Metric
- C12, C13, C25, C28, C30, C31, C34, C35, C36, C37, C38, C39, C55, C56, C59, C60, C62: footprint Capacitor_SMD:C_0603_1608Metric -> Capacitor_SMD:C_0402_1005Metric
- C14, C42: footprint Capacitor_SMD:C_1206_3216Metric_Pad1.33x1.80mm_HandSolder -> Capacitor_SMD:C_0603_1608Metric
- C27, C3, C4, C5: footprint Capacitor_SMD:C_0805_2012Metric_Pad1.18x1.45mm_HandSolder -> Capacitor_SMD:C_0603_1608Metric
- C29: footprint Capacitor_SMD:C_0805_2012Metric_Pad1.18x1.45mm_HandSolder -> Capacitor_SMD:C_0402_1005Metric
- C32, C33, C7: footprint Capacitor_SMD:C_0603_1608Metric_Pad1.08x0.95mm_HandSolder -> Capacitor_SMD:C_0402_1005Metric
- C53, C58: footprint Capacitor_SMD:C_0603_1608Metric -> Capacitor_SMD:C_0402_1005Metric; moved to B.Cu
- C57: footprint Capacitor_SMD:C_1206_3216Metric_Pad1.33x1.80mm_HandSolder -> Capacitor_SMD:C_0603_1608Metric; moved to B.Cu
- C6, C8, C9: footprint Capacitor_SMD:C_0603_1608Metric_Pad1.08x0.95mm_HandSolder -> Capacitor_SMD:C_0603_1608Metric
- D1, D14, D17, D3: footprint LED_SMD:LED_0603_1608Metric_Pad1.05x0.95mm_HandSolder -> LED_SMD:LED_0402_1005Metric
- D10, D11, D4, D5, D6, D7, D8, D9: footprint LED_SMD:LED_0805_2012Metric_Pad1.15x1.40mm_HandSolder -> LED_SMD:LED_0402_1005Metric
- FB1, FB2: footprint Inductor_SMD:L_0805_2012Metric_Pad1.05x1.20mm_HandSolder -> Inductor_SMD:L_0402_1005Metric
- FB3, FB4, FB5, FB6: footprint Inductor_SMD:L_0805_2012Metric_Pad1.05x1.20mm_HandSolder -> Inductor_SMD:L_0603_1608Metric
- L2: footprint Inductor_SMD:L_0603_1608Metric_Pad1.05x0.95mm_HandSolder -> Inductor_SMD:L_0402_1005Metric
- R10, R11, R12, R13, R14, R19, R20, R21, R22, R23, R24, R25, R26, R27, R28, R29, R3, R30, R31, R32, R33, R34, R4, R49, R53, R8, R9: footprint Resistor_SMD:R_0603_1608Metric_Pad0.98x0.95mm_HandSolder -> Resistor_SMD:R_0402_1005Metric
- R15, R16, R17, R18, R46, R47, R48, R50, R51, R52: footprint Resistor_SMD:R_0603_1608Metric_Pad0.98x0.95mm_HandSolder -> Resistor_SMD:R_0402_1005Metric; moved to F.Cu
- R35, R36, R37, R38, R39, R40, R41, R42, R43, R44: footprint Resistor_SMD:R_0402_1005Metric_Pad0.72x0.64mm_HandSolder -> Resistor_SMD:R_0402_1005Metric
- R54: footprint Resistor_SMD:R_0603_1608Metric_Pad0.98x0.95mm_HandSolder -> Resistor_SMD:R_0402_1005Metric; moved to B.Cu
- moved TP4 110.0 mm to (279.4, 100.8)
- moved TP3 107.1 mm to (279.4, 97.8)
- moved R11 106.1 mm to (76.1, 110.2), turned to 0 degrees
- moved C11 98.6 mm to (89.5, 26.1)
- moved C2 98.6 mm to (89.5, 22.7)
- moved R1 96.0 mm to (84.5, 22.3)
- moved U9 95.0 mm to (73.4, 77.9)
- moved C13 90.2 mm to (67.5, 106.2)
- moved SW1 90.0 mm to (247.9, 137.3), turned to 90 degrees
- moved D3 89.6 mm to (84.0, 34.0)
- moved C36 88.6 mm to (85.2, 74.8), turned to 0 degrees
- moved R8 87.1 mm to (95.7, 32.7)
- moved C12 86.5 mm to (67.5, 104.3), turned to 0 degrees
- moved C19 86.3 mm to (70.3, 106.2), turned to 0 degrees
- moved JP2 85.8 mm to (37.2, 93.9), turned to 0 degrees
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Other:
- board size 106.1 x 55 mm -> 100 x 50 mm
- board text removed: "100x55"
- board text removed: "C O M"
- board text removed: "F L H"
- board text removed: "FlyCU"
- board text removed: "GravitumFCS"
- board text removed: "Made by Breno Soares Alves"
- board text removed: "P W R"
- board text removed: "S T S"
- board text removed: "SCL"
- board text removed: "SDA"
