File: hardware/flight_control_unit.kicad_sch (KiCad schematic)
At the start: 36 parts, among them SW4 SW_Push_Dual, SW5 SW_SPDT_312, SW6 SW_SPDT_312, U8 STM32F405RGTx, Y2 25MHz

Commit message: schematic and BOM done
Parts:
- removed C29: 10u, symbol Device:C_Polarized
- added C29: 10u, Capacitor_SMD:C_0603_1608Metric, symbol Device:C
- C27, C28: footprint (none) -> Capacitor_SMD:C_0805_2012Metric
- C30, C34: value 10p -> 25p; footprint (none) -> Capacitor_SMD:C_0603_1608Metric
- C31, C32, C33, C35, C36, C37, C38: footprint (none) -> Capacitor_SMD:C_0402_1005Metric
- C39: footprint (none) -> Capacitor_SMD:C_0603_1608Metric
- D10, D6, D7, D8, D9: footprint (none) -> LED_SMD:LED_0603_1608Metric
- FB2: footprint (none) -> Inductor_SMD:L_0603_1608Metric
- R15, R16, R17, R21, R22, R23, R24, R25, R26: footprint (none) -> Resistor_SMD:R_0603_1608Metric
- R18, R19: value 560 -> 100; footprint (none) -> Resistor_SMD:R_0603_1608Metric
- R20: value R -> 620; footprint (none) -> Resistor_SMD:R_0603_1608Metric
- SW4: footprint (none) -> airplane:SW_TL3365AF180QG; Manufacturer Part Number (none) -> TL3365AF180QG
- SW5, SW6: footprint (none) -> Button_Switch_SMD:SW_SPDT_PCM12; Manufacturer Part Number (none) -> PCM12SMTR
- U8: Manufacturer Part Number (none) -> STM32F405RGT6
- Y2: footprint (none) -> airplane:XTAL_ABM8G-25.000MHZ-18-D2Y-T; Manufacturer Part Number (none) -> ABM8G-25.000MHZ-18-D2Y-T
Connections:
- net +3.3V: now also C29.1
- net GND: now also C29.2
- net USB_OTG_FS_D+ renamed FCU_USB_OTG_FS_D+
- net USB_OTG_FS_D- renamed FCU_USB_OTG_FS_D-
- net USB_OTG_FS_ID renamed FCU_USB_OTG_FS_ID
- net USB_OTG_FS_VBUS renamed FCU_USB_OTG_FS_VBUS
